File: boards/opAmp1/opAmp1.sch (KiCad schematic (older format))
At the start: 23 parts, among them P1 CONN_01X02, P2 CONN_01X02, P3 CONN_01X02, Q1 TIP122, Q2 BC817-40, U1 LM324N, U2 TL431_SOT23-3

Commit message: design of test platform, opAmp idea, refinements
Parts:
- renumbered C2 to C?, C7 to C?, C6 to C?, C5 to C?, C3 to C?, C8 to C?, C4 to C?
Changed lines of the file:
@@
 $EndComp
 $Comp
-L GND #PWR8
+L GND #PWR01
 U 1 1 552D5DD3
 P 5350 4650
-F 0 "#PWR8" H 5350 4400 60  0001 C CNN
+F 0 "#PWR01" H 5350 4400 60  0001 C CNN
 F 1 "GND" H 5350 4500 60  0000 C CNN
 F 2 "" H 5350 4650 60  0000 C CNN
@@
 $EndComp
 $Comp
-L +24V #PWR1
+L +24V #PWR02
 U 1 1 552D5DF7
 P 5350 2200
-F 0 "#PWR1" H 5350 2050 60  0001 C CNN
+F 0 "#PWR02" H 5350 2050 60  0001 C CNN
 F 1 "+24V" H 5350 2340 60  0000 C CNN
 F 2 "" H 5350 2200 60  0000 C CNN
@@
 $EndComp
 $Comp
-L GND #PWR7
+L GND #PWR03
 U 1 1 552D68DB
 P 7300 4000
-F 0 "#PWR7" H 7300 3750 60  0001 C CNN
+F 0 "#PWR03" H 7300 3750 60  0001 C CNN
 F 1 "GND" H 7300 3850 60  0000 C CNN
 F 2 "" H 7300 4000 60  0000 C CNN
@@
 	6900 3700 6900 4600
 $Comp
-L GND #PWR9
+L GND #PWR04
 U 1 1 552D7112
 P 8000 5000
-F 0 "#PWR9" H 8000 4750 60  0001 C CNN
+F 0 "#PWR04" H 8000 4750 60  0001 C CNN
 F 1 "GND" H 8000 4850 60  0000 C CNN
 F 2 "" H 8000 5000 60  0000 C CNN
@@
 	7300 2750 7300 3200
 $Comp
-L GND #PWR4
+L GND #PWR05
 U 1 1 552D8314
 P 7700 3000
-F 0 "#PWR4" H 7700 2750 60  0001 C CNN
+F 0 "#PWR05" H 7700 2750 60  0001 C CNN
 F 1 "GND" H 7700 2850 60  0000 C CNN
 F 2 "" H 7700 3000 60  0000 C CNN
@@
 $EndComp
 $Comp
-L GND #PWR6
+L GND #PWR06
 U 1 1 552D8A33
 P 3650 3600
-F 0 "#PWR6" H 3650 3350 60  0001 C CNN
+F 0 "#PWR06" H 3650 3350 60  0001 C CNN
 F 1 "GND" H 3650 3450 60  0000 C CNN
 F 2 "" H 3650 3600 60  0000 C CNN
@@
 Connection ~ 4350 2250
 $Comp
-L GND #PWR2
+L GND #PWR07
 U 1 1 552D8F95
 P 2900 2400
-F 0 "#PWR2" H 2900 2150 60  0001 C CNN
+F 0 "#PWR07" H 2900 2150 60  0001 C CNN
 F 1 "GND" H 2900 2250 60  0000 C CNN
 F 2 "" H 2900 2400 60  0000 C CNN
@@
 	2500 3400 2850 3400
 $Comp
-L GND #PWR5
+L GND #PWR08
 U 1 1 552D912D
 P 2500 3500
-F 0 "#PWR5" H 2500 3250 60  0001 C CNN
+F 0 "#PWR08" H 2500 3250 60  0001 C CNN
 F 1 "GND" H 2500 3350 60  0000 C CNN
 F 2 "" H 2500 3500 60  0000 C CNN
@@
 Connection ~ 7300 2950
 $Comp
-L PWR_FLAG #FLG3
+L PWR_FLAG #FLG09
 U 1 1 552D9604
 P 7300 2950
-F 0 "#FLG3" H 7300 3045 30  0001 C CNN
+F 0 "#FLG09" H 7300 3045 30  0001 C CNN
 F 1 "PWR_FLAG" H 7300 3130 30  0000 C CNN
 F 2 "" H 7300 2950 60  0000 C CNN
@@
 $EndComp
 $Comp
-L PWR_FLAG #FLG1
+L PWR_FLAG #FLG010
 U 1 1 552D97E2
 P 2650 2200
-F 0 "#FLG1" H 2650 2295 30  0001 C CNN
+F 0 "#FLG010" H 2650 2295 30  0001 C CNN
 F 1 "PWR_FLAG" H 2650 2380 30  0000 C CNN
 F 2 "" H 2650 2200 60  0000 C CNN
@@
 $EndComp
 $Comp
-L PWR_FLAG #FLG2
+L PWR_FLAG #FLG011
 U 1 1 552D9857
 P 2650 2450
-F 0 "#FLG2" H 2650 2545 30  0001 C CNN
+F 0 "#FLG011" H 2650 2545 30  0001 C CNN
 F 1 "PWR_FLAG" H 2650 2630 30  0000 C CNN
 F 2 "" H 2650 2450 60  0000 C CNN
@@
 100n*20k = 2ms\nSoft-start, but aren't\nany oscillations introduced?
 $Comp
-L C C2
+L C C?
 U 1 1 552E6250
 P 3150 2400
-F 0 "C2" H 3175 2500 50  0000 L CNN
+F 0 "C?" H 3175 2500 50  0000 L CNN
 F 1 "1n" H 3175 2300 50  0000 L CNN
 F 2 "Capacitors_SMD:C_0805_HandSoldering" H 4000 2750 30  0000 C CNN
@@
 1nF here is for decoupling\nhigh-frequency garbage\nfrom LED leads. Is it better\nto have 100nF, 1uF or 100uF\nhere (stability)? Why?
 $Comp
-L C C7
+L C C?
 U 1 1 552E6251
 P 5100 2700
-F 0 "C7" H 5125 2800 50  0000 L CNN
+F 0 "C?" H 5125 2800 50  0000 L CNN
 F 1 "1n" H 5125 2600 50  0000 L CNN
 F 2 "Capacitors_SMD:C_0805_HandSoldering" H 5800 3000 30  0000 C CNN
@@
 $EndComp
 $Comp
-L GND #PWR3
+L GND #PWR?
 U 1 1 552E6252
 P 3400 2550
-F 0 "#PWR3" H 3400 2300 60  0001 C CNN
+F 0 "#PWR?" H 3400 2300 60  0001 C CNN
 F 1 "GND" H 3400 2400 60  0000 C CNN
 F 2 "" H 3400 2550 60  0000 C CNN
@@
 1nF here is for decoupling\nhigh-frequency garbage\nfrom input. Some reason\nto have 100nF, 1uF or 100uF\nin such low freq. design?
 $Comp
-L C C6
+L C C?
 U 1 1 552E6253
 P 4850 2700
-F 0 "C6" H 4875 2800 50  0000 L CNN
+F 0 "C?" H 4875 2800 50  0000 L CNN
 F 1 "100n" H 4875 2600 50  0000 L CNN
 F 2 "Capacitors_SMD:C_0805_HandSoldering" H 5800 3050 30  0000 C CNN
@@
 $EndComp
 $Comp
-L CP C5
+L CP C?
 U 1 1 552E6254
 P 4600 2700
-F 0 "C5" H 4625 2800 50  0000 L CNN
+F 0 "C?" H 4625 2800 50  0000 L CNN
 F 1 "1u" H 4625 2600 50  0000 L CNN
 F 2 "Capacitors_Elko_ThroughHole:Elko_vert_11.2x7.5mm_RM2.5_CopperClear" H 5900 2950 20  0000 C CNN
@@
 Connection ~ 5350 2550
 $Comp
-L C C3
+L C C?
 U 1 1 552E9E96
 P 3400 2400
-F 0 "C3" H 3425 2500 50  0000 L CNN
+F 0 "C?" H 3425 2500 50  0000 L CNN
 F 1 "100n" H 3425 2300 50  0000 L CNN
 F 2 "Capacitors_SMD:C_0805_HandSoldering" H 4000 2700 30  0000 C CNN
@@
 	3150 2550 3650 2550
 $Comp
-L C C8
+L C C?
 U 1 1 552EA8C7
 P 4900 3900
-F 0 "C8" H 4925 4000 50  0000 L CNN
+F 0 "C?" H 4925 4000 50  0000 L CNN
 F 1 "100n" H 4925 3800 50  0000 L CNN
 F 2 "Capacitors_SMD:C_0805_HandSoldering" V 4750 3900 30  0000 C CNN
@@
 Connection ~ 4900 4600
 $Comp
-L CP C4
+L CP C?
 U 1 1 552EC3CD
 P 3650 2400
-F 0 "C4" H 3675 2500 50  0000 L CNN
+F 0 "C?" H 3675 2500 50  0000 L CNN
 F 1 "1u" H 3675 2300 50  0000 L CNN
 F 2 "Capacitors_Elko_ThroughHole:Elko_vert_11.2x7.5mm_RM2.5_CopperClear" H 4100 2650 20  0000 C CNN

Commit message: designing
Parts:
- removed C1: 100n, symbol C
- removed R3, R6: 1k, Resistors_SMD:R_0805_HandSoldering, symbol R
- removed R5: 20k, Resistors_SMD:R_0805_HandSoldering, symbol R
- removed RV1: 100k, symbol POT
- removed U1: LM324N, Housings_SOIC:SOIC-14_3.9x8.7mm_Pitch1.27mm, symbol LM324N
- removed U2: TL431_SOT23-3, Housings_SOT-23_SOT-143_TSOT-6:SOT-23_Handsoldering, symbol TL431_SOT23-3
- added C?: 100nF, symbol C_Small
- added Q?: Q_NPN_BCE, symbol Q_NPN_BCE
- added R?: 2k, symbol R
- added R? (x2): 100R, symbol R
- added R? (x2): 3k3, symbol R
- added R? (x2): 100k, symbol R
- added R? (x2): 4k7, symbol R
- added R? (x2): 20k, symbol R
- added U? (x2): LM324N, symbol LM324N
Connections:
- wire segments 41 -> 65
Other:
- note added: "0-4.125 V ref.\nZout << 4k7"
- note added: "10mA more -> 33mV diff\n-> 660mV diff"
- note added: "21x gain differential amplifier"
- note added: "3.3V / 1A"
- note added: "33x gain differential amplifier"
- note added: "3k3 and 100R is tuned\nto minimize I_offset error."
- note added: "How to study stability?"
- note added: "LED OUT\nwhich output capacitors are required?"
- note added: "to minimize 0-2.5V reference\noutput impedance error"
- note removed: "100R * 1e-7F =\n= 1e-5s = 10us"
- note removed: "20x - 120x gain -> 1.25A - 0.2A"
- moved on the sheet: C?, P1, P2, P3, Q1, Q2, R1, R2, R4, R7

Commit message: upgrade
Parts:
- removed Q1: TIP122, Transistors_TO-220:TO-220_Bipolar-BCE_Horizontal_MountedFromLS_LargePads, symbol TIP122
- removed R?: 20k, symbol R
- added Q1: TIP127, TO-220, symbol TIP127
- added R17: 20k, symbol R
- added R3: 10k, Resistors_SMD:R_0805_HandSoldering, symbol R
- added R5: 1k, Resistors_SMD:R_0805_HandSoldering, symbol R
- C5: renamed from C?; footprint (none) -> Capacitors_SMD:C_0805_HandSoldering
- R12, R14, R15, R6, R9: renamed from R?; footprint (none) -> Resistors_SMD:R_0805_HandSoldering
- R13: renamed from R?; value 2k -> 4k7; footprint (none) -> Resistors_SMD:R_0805_HandSoldering
- R2: value 1k -> 4k7
- gave numbers to parts that had none: 13
Connections:
- net labels added: +5V
- wire segments 65 -> 92
Other:
- note added: "1/11 divider\n(24V -> 2.18V,\n 27.5 -> 2.5V)"
- note added: "10mA more -> 33mV diff\n-> 700mV diff"
- note added: "8k 120R"
- note added: "TIP127 hFE ca 4000@1A,25C"
- note removed: "10mA more -> 33mV diff\n-> 660mV diff"
- note removed: "COLLECTOR CUTOFF CURRENT\nI_CE0 < 0.5 mA\nhow much it is?\nit will light-up high-power LEDs?"
- note removed: "How to study stability?"
- note removed: "LED OUT\nwhich output capacitors are required?"
- note removed: "TIP122: h_FE>3000 @ 1.25A\n2 mA * 24 V < 50 mW"
- note removed: "V_CEsat. < 0.8V"
- note removed: "What is load and line regulation?\nCan this design start oscillate somehow??"
- moved on the sheet: C1, C2, C3, C4, C5, C6, C7, C8, P1, P2, P3, Q2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
